Commit message: Tried to fix urdf

File: arm_ws/install/FINAL_description/share/FINAL_description/urdf/FINAL.xacro (robot description, xacro)
@@ -13,5 +13,5 @@
     <origin xyz="0 0 0" rpy="0 0 0"/>
     <geometry>
-      <mesh filename="file://$(find FINAL_description)/meshes/base_link.stl" scale="0.001 0.001 0.001"/>
+      <mesh filename="$(find FINAL_description)/meshes/base_link.stl" scale="0.001 0.001 0.001"/>
     </geometry>
     <material name="silver"/>
@@ -20,5 +20,5 @@
     <origin xyz="0 0 0" rpy="0 0 0"/>
     <geometry>
-      <mesh filename="file://$(find FINAL_description)/meshes/base_link.stl" scale="0.001 0.001 0.001"/>
+      <mesh filename="$(find FINAL_description)/meshes/base_link.stl" scale="0.001 0.001 0.001"/>
     </geometry>
   </collision>
@@ -33,5 +33,5 @@
     <origin xyz="-0.0075 -0.1025 0.037395" rpy="0 0 0"/>
     <geometry>
-      <mesh filename="file://$(find FINAL_description)/meshes/Sun_Connector_Shaft,_0.2497''_1.stl" scale="0.001 0.001 0.001"/>
+      <mesh filename="$(find FINAL_description)/meshes/Sun_Connector_Shaft,_0.2497''_1.stl" scale="0.001 0.001 0.001"/>
     </geometry>
     <material name="silver"/>
@@ -40,5 +40,5 @@
     <origin xyz="-0.0075 -0.1025 0.037395" rpy="0 0 0"/>
     <geometry>
-      <mesh filename="file://$(find FINAL_description)/meshes/Sun_Connector_Shaft,_0.2497''_1.stl" scale="0.001 0.001 0.001"/>
+      <mesh filename="$(find FINAL_description)/meshes/Sun_Connector_Shaft,_0.2497''_1.stl" scale="0.001 0.001 0.001"/>
     </geometry>
   </collision>
@@ -53,5 +53,5 @@
     <origin xyz="-0.0075 -0.1025 0.006915" rpy="0 0 0"/>
     <geometry>
-      <mesh filename="file://$(find FINAL_description)/meshes/Planetary_Gear_Arm_Connector,1_1.stl" scale="0.001 0.001 0.001"/>
+      <mesh filename="$(find FINAL_description)/meshes/Planetary_Gear_Arm_Connector,1_1.stl" scale="0.001 0.001 0.001"/>
     </geometry>
     <material name="silver"/>
@@ -60,5 +60,5 @@
     <origin xyz="-0.0075 -0.1025 0.006915" rpy="0 0 0"/>
     <geometry>
-      <mesh filename="file://$(find FINAL_description)/meshes/Planetary_Gear_Arm_Connector,1_1.stl" scale="0.001 0.001 0.001"/>
+      <mesh filename="$(find FINAL_description)/meshes/Planetary_Gear_Arm_Connector,1_1.stl" scale="0.001 0.001 0.001"/>
     </geometry>
   </collision>
@@ -73,5 +73,5 @@
     <origin xyz="-0.0075 -0.1025 0.005137" rpy="0 0 0"/>
     <geometry>
-      <mesh filename="file://$(find FINAL_description)/meshes/Arm_1_1.stl" scale="0.001 0.001 0.001"/>
+      <mesh filename="$(find FINAL_description)/meshes/Arm_1_1.stl" scale="0.001 0.001 0.001"/>
     </geometry>
     <material name="silver"/>
@@ -80,5 +80,5 @@
     <origin xyz="-0.0075 -0.1025 0.005137" rpy="0 0 0"/>
     <geometry>
-      <mesh filename="file://$(find FINAL_description)/meshes/Arm_1_1.stl" scale="0.001 0.001 0.001"/>
+      <mesh filename="$(find FINAL_description)/meshes/Arm_1_1.stl" scale="0.001 0.001 0.001"/>
     </geometry>
   </collision>
@@ -93,5 +93,5 @@
     <origin xyz="-0.0295 -0.1025 -0.153863" rpy="0 0 0"/>
     <geometry>
-      <mesh filename="file://$(find FINAL_description)/meshes/Gear_1_1.stl" scale="0.001 0.001 0.001"/>
+      <mesh filename="$(find FINAL_description)/meshes/Gear_1_1.stl" scale="0.001 0.001 0.001"/>
     </geometry>
     <material name="silver"/>
@@ -100,5 +100,5 @@
     <origin xyz="-0.0295 -0.1025 -0.153863" rpy="0 0 0"/>
     <geometry>
-      <mesh filename="file://$(find FINAL_description)/meshes/Gear_1_1.stl" scale="0.001 0.001 0.001"/>
+      <mesh filename="$(find FINAL_description)/meshes/Gear_1_1.stl" scale="0.001 0.001 0.001"/>
     </geometry>
   </collision>
@@ -113,5 +113,5 @@
     <origin xyz="-0.0295 -0.1025 -0.518363" rpy="0 0 0"/>
     <geometry>
-      <mesh filename="file://$(find FINAL_description)/meshes/Gear_3,_UPDATED_1.stl" scale="0.001 0.001 0.001"/>
+      <mesh filename="$(find FINAL_description)/meshes/Gear_3,_UPDATED_1.stl" scale="0.001 0.001 0.001"/>
     </geometry>
     <material name="silver"/>
@@ -120,5 +120,5 @@
     <origin xyz="-0.0295 -0.1025 -0.518363" rpy="0 0 0"/>
     <geometry>
-      <mesh filename="file://$(find FINAL_description)/meshes/Gear_3,_UPDATED_1.stl" scale="0.001 0.001 0.001"/>
+      <mesh filename="$(find FINAL_description)/meshes/Gear_3,_UPDATED_1.stl" scale="0.001 0.001 0.001"/>
     </geometry>
   </collision>
@@ -133,5 +133,5 @@
     <origin xyz="-0.4145 -0.1025 -0.518363" rpy="0 0 0"/>
     <geometry>
-      <mesh filename="file://$(find FINAL_description)/meshes/Manipulator3__2__1.stl" scale="0.001 0.001 0.001"/>
+      <mesh filename="$(find FINAL_description)/meshes/Manipulator3__2__1.stl" scale="0.001 0.001 0.001"/>
     </geometry>
     <material name="silver"/>
@@ -140,5 +140,5 @@
     <origin xyz="-0.4145 -0.1025 -0.518363" rpy="0 0 0"/>
     <geometry>
-      <mesh filename="file://$(find FINAL_description)/meshes/Manipulator3__2__1.stl" scale="0.001 0.001 0.001"/>
+      <mesh filename="$(find FINAL_description)/meshes/Manipulator3__2__1.stl" scale="0.001 0.001 0.001"/>
     </geometry>
   </collision>
