Commit message: Overrode arm workspace

File: arm_ws/install/FINAL_description/share/FINAL_description/urdf/FINAL.urdf (robot description, URDF)
Before this commit: robot FINAL, 7 links, 6 joints
Links:
- removed link Sun_Connector_Shaft,_0.2497''_1
- added link sun_connector_shaft_1, mass 0.007456676389725328; collision mesh filename=$(find FINAL_description)/meshes/Sun_Connector_Shaft,_0.249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 scale=0.001 0.001 0.001; visual mesh filename=$(find FINAL_description)/meshes/Sun_Connector_Shaft,_0.249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 scale=0.001 0.001 0.001
- added link world
- link Arm_1_1: geometry collision mesh filename=$(find FINAL_description)/meshes/Arm_1_1.stl scale=0.001 0.001 0.001; visual mesh filename=$(find FINAL_description)/meshes/Arm_1_1.stl scale=0.001 0.001 0.001
- link Gear_1_1: geometry collision mesh filename=$(find FINAL_description)/meshes/Gear_1_1.stl scale=0.001 0.001 0.001; visual mesh filename=$(find FINAL_description)/meshes/Gear_1_1.stl scale=0.001 0.001 0.001
- link Gear_3,_UPDATED_1: geometry collision mesh filename=$(find FINAL_description)/meshes/Gear_3,_UPDATED_1.stl scale=0.001 0.001 0.001; visual mesh filename=$(find FINAL_description)/meshes/Gear_3,_UPDATED_1.stl scale=0.001 0.001 0.001
- link Manipulator3__2__1: geometry collision mesh filename=$(find FINAL_description)/meshes/Manipulator3__2__1.stl scale=0.001 0.001 0.001; visual mesh filename=$(find FINAL_description)/meshes/Manipulator3__2__1.stl scale=0.001 0.001 0.001
- link Planetary_Gear_Arm_Connector,1_1: geometry collision mesh filename=$(find FINAL_description)/meshes/Planetary_Gear_Arm_Connect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 scale=0.001 0.001 0.001; visual mesh filename=$(find FINAL_description)/meshes/Planetary_Gear_Arm_Connect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 scale=0.001 0.001 0.001
- link base_link: mass 0.4973707256934835 -> 1.0; geometry collision mesh filename=$(find FINAL_description)/meshes/base_link.stl scale=0.001 0.001 0.001; visual mesh filename=$(find FINAL_description)/meshes/base_link.stl scale=0.001 0.001 0.001
Joints:
- added joint world_to_base: type fixed, parent world, child base_link, origin xyz=0 0 .1 rpy=0 0 0
- joint Revolute 40: child Sun_Connector_Shaft,_0.2497''_1 -> sun_connector_shaft_1
- joint Rigid 41: parent Sun_Connector_Shaft,_0.2497''_1 -> sun_connector_shaft_1

File: arm_ws/install/FINAL_description/share/FINAL_description/urdf/FINAL.xacro (robot description, xacro)
@@ -4,10 +4,19 @@
 <xacro:include filename="$(find FINAL_description)/urdf/FINAL.trans" />
 <xacro:include filename="$(find FINAL_description)/urdf/FINAL.gazebo" />
+<material name="grey">
+        <color rgba="0.7 0.7 0.7 1"/>
+    </material>
+<link name="world"></link>
+<joint name="world_to_base" type="fixed">
+        <parent link="world" />
+        <child link="base_link" />
+        <origin  rpy="0 0 0" xyz="0 0 .1" />
+    </joint>
 <link name="base_link">
-  <inertial>
-    <origin xyz="0.09585265642198176 0.11340397705901449 0.23015193841971182" rpy="0 0 0"/>
-    <mass value="0.4973707256934835"/>
-    <inertia ixx="0.000128" iyy="0.000132" izz="0.000128" ixy="-0.0" iyz="-1e-06" ixz="-4e-06"/>
-  </inertial>
+<inertial>
+            <mass value="1.0"/>
+            <origin xyz="0 0 0"/>
+            <inertia ixx="0.1" ixy="0.0" ixz="0.0" iyy="0.1" iyz="0.0" izz="0.1"/>
+        </inertial>
   <visual>
     <origin xyz="0 0 0" rpy="0 0 0"/>
@@ -15,5 +24,5 @@
       <mesh filename="$(find FINAL_description)/meshes/base_link.stl" scale="0.001 0.001 0.001"/>
     </geometry>
-    <material name="silver"/>
+    <material name="grey"/>
   </visual>
   <collision>
@@ -24,5 +33,5 @@
   </collision>
 </link>
-<link name="Sun_Connector_Shaft,_0.2497''_1">
+<link name="sun_connector_shaft_1">
   <inertial>
     <origin xyz="3.290622982432545e-13 -9.536743103555345e-09 0.0152396655965897" rpy="0 0 0"/>
@@ -35,5 +44,5 @@
       <mesh filename="$(find FINAL_description)/meshes/Sun_Connector_Shaft,_0.2497''_1.stl" scale="0.001 0.001 0.001"/>
     </geometry>
-    <material name="silver"/>
+    <material name="grey"/>
   </visual>
   <collision>
@@ -55,5 +64,5 @@
       <mesh filename="$(find FINAL_description)/meshes/Planetary_Gear_Arm_Connector,1_1.stl" scale="0.001 0.001 0.001"/>
     </geometry>
-    <material name="silver"/>
+    <material name="grey"/>
   </visual>
   <collision>
@@ -75,5 +84,5 @@
       <mesh filename="$(find FINAL_description)/meshes/Arm_1_1.stl" scale="0.001 0.001 0.001"/>
     </geometry>
-    <material name="silver"/>
+    <material name="grey"/>
   </visual>
   <collision>
@@ -95,5 +104,5 @@
       <mesh filename="$(find FINAL_description)/meshes/Gear_1_1.stl" scale="0.001 0.001 0.001"/>
     </geometry>
-    <material name="silver"/>
+    <material name="grey"/>
   </visual>
   <collision>
@@ -115,5 +124,5 @@
       <mesh filename="$(find FINAL_description)/meshes/Gear_3,_UPDATED_1.stl" scale="0.001 0.001 0.001"/>
     </geometry>
-    <material name="silver"/>
+    <material name="grey"/>
   </visual>
   <collision>
@@ -135,5 +144,5 @@
       <mesh filename="$(find FINAL_description)/meshes/Manipulator3__2__1.stl" scale="0.001 0.001 0.001"/>
     </geometry>
-    <material name="silver"/>
+    <material name="grey"/>
   </visual>
   <collision>
@@ -147,10 +156,10 @@
   <origin xyz="0.0075 0.1025 -0.037395" rpy="0 0 0"/>
   <parent link="base_link"/>
-  <child link="Sun_Connector_Shaft,_0.2497''_1"/>
+  <child link="sun_connector_shaft_1"/>
   <axis xyz="-0.0 0.0 1.0"/>
 </joint>
 <joint name="Rigid 41" type="fixed">
   <origin xyz="0.0 0.0 0.03048" rpy="0 0 0"/>
-  <parent link="Sun_Connector_Shaft,_0.2497''_1"/>
+  <parent link="sun_connector_shaft_1"/>
   <child link="Planetary_Gear_Arm_Connector,1_1"/>
 </joint>
