Commit message: Updated  FINAL.xacro mesh tags

File: arm_ws/src/FINAL_description/urdf/FINAL.xacro (robot description, xacro)
@@ -1,7 +1,7 @@
 <?xml version="1.0" ?>
 <robot name="FINAL" xmlns:xacro="http://www.ros.org/wiki/xacro">
-<xacro:include filename="$(find FINAL_description)/urdf/materials.xacro" />
-<xacro:include filename="$(find FINAL_description)/urdf/FINAL.trans" />
-<xacro:include filename="$(find FINAL_description)/urdf/FINAL.gazebo" />
+<xacro:include filename="materials.xacro" />
+<xacro:include filename="FINAL.trans" />
+<xacro:include filename="FINAL.gazebo" />
 <material name="grey">
         <color rgba="0.7 0.7 0.7 1"/>
@@ -22,5 +22,5 @@
     <origin xyz="0 0 0" rpy="0 0 0"/>
     <geometry>
-      <mesh filename="$(find FINAL_description)/meshes/base_link.stl" scale="0.001 0.001 0.001"/>
+      <mesh filename="package://FINAL_description/meshes/base_link.stl" scale="0.001 0.001 0.001"/>
     </geometry>
     <material name="grey"/>
@@ -29,5 +29,5 @@
     <origin xyz="0 0 0" rpy="0 0 0"/>
     <geometry>
-      <mesh filename="$(find FINAL_description)/meshes/base_link.stl" scale="0.001 0.001 0.001"/>
+      <mesh filename="package://FINAL_description/meshes/base_link.stl" scale="0.001 0.001 0.001"/>
     </geometry>
   </collision>
@@ -42,5 +42,5 @@
     <origin xyz="-0.0075 -0.1025 0.037395" rpy="0 0 0"/>
     <geometry>
-      <mesh filename="$(find FINAL_description)/meshes/Sun_Connector_Shaft,_0.2497''_1.stl" scale="0.001 0.001 0.001"/>
+      <mesh filename="package://FINAL_description/meshes/Sun_Connector_Shaft,_0.2497''_1.stl" scale="0.001 0.001 0.001"/>
     </geometry>
     <material name="grey"/>
@@ -49,5 +49,5 @@
     <origin xyz="-0.0075 -0.1025 0.037395" rpy="0 0 0"/>
     <geometry>
-      <mesh filename="$(find FINAL_description)/meshes/Sun_Connector_Shaft,_0.2497''_1.stl" scale="0.001 0.001 0.001"/>
+      <mesh filename="package://FINAL_description/meshes/Sun_Connector_Shaft,_0.2497''_1.stl" scale="0.001 0.001 0.001"/>
     </geometry>
   </collision>
@@ -62,5 +62,5 @@
     <origin xyz="-0.0075 -0.1025 0.006915" rpy="0 0 0"/>
     <geometry>
-      <mesh filename="$(find FINAL_description)/meshes/Planetary_Gear_Arm_Connector,1_1.stl" scale="0.001 0.001 0.001"/>
+      <mesh filename="package://FINAL_description/meshes/Planetary_Gear_Arm_Connector,1_1.stl" scale="0.001 0.001 0.001"/>
     </geometry>
     <material name="grey"/>
@@ -69,5 +69,5 @@
     <origin xyz="-0.0075 -0.1025 0.006915" rpy="0 0 0"/>
     <geometry>
-      <mesh filename="$(find FINAL_description)/meshes/Planetary_Gear_Arm_Connector,1_1.stl" scale="0.001 0.001 0.001"/>
+      <mesh filename="package://FINAL_description/meshes/Planetary_Gear_Arm_Connector,1_1.stl" scale="0.001 0.001 0.001"/>
     </geometry>
   </collision>
@@ -82,5 +82,5 @@
     <origin xyz="-0.0075 -0.1025 0.005137" rpy="0 0 0"/>
     <geometry>
-      <mesh filename="$(find FINAL_description)/meshes/Arm_1_1.stl" scale="0.001 0.001 0.001"/>
+      <mesh filename="package://FINAL_description/meshes/Arm_1_1.stl" scale="0.001 0.001 0.001"/>
     </geometry>
     <material name="grey"/>
@@ -89,5 +89,5 @@
     <origin xyz="-0.0075 -0.1025 0.005137" rpy="0 0 0"/>
     <geometry>
-      <mesh filename="$(find FINAL_description)/meshes/Arm_1_1.stl" scale="0.001 0.001 0.001"/>
+      <mesh filename="package://FINAL_description/meshes/Arm_1_1.stl" scale="0.001 0.001 0.001"/>
     </geometry>
   </collision>
@@ -102,5 +102,5 @@
     <origin xyz="-0.0295 -0.1025 -0.153863" rpy="0 0 0"/>
     <geometry>
-      <mesh filename="$(find FINAL_description)/meshes/Gear_1_1.stl" scale="0.001 0.001 0.001"/>
+      <mesh filename="package://FINAL_description/meshes/Gear_1_1.stl" scale="0.001 0.001 0.001"/>
     </geometry>
     <material name="grey"/>
@@ -109,5 +109,5 @@
     <origin xyz="-0.0295 -0.1025 -0.153863" rpy="0 0 0"/>
     <geometry>
-      <mesh filename="$(find FINAL_description)/meshes/Gear_1_1.stl" scale="0.001 0.001 0.001"/>
+      <mesh filename="package://FINAL_description/meshes/Gear_1_1.stl" scale="0.001 0.001 0.001"/>
     </geometry>
   </collision>
@@ -122,5 +122,5 @@
     <origin xyz="-0.0295 -0.1025 -0.518363" rpy="0 0 0"/>
     <geometry>
-      <mesh filename="$(find FINAL_description)/meshes/Gear_3,_UPDATED_1.stl" scale="0.001 0.001 0.001"/>
+      <mesh filename="package://FINAL_description/meshes/Gear_3,_UPDATED_1.stl" scale="0.001 0.001 0.001"/>
     </geometry>
     <material name="grey"/>
@@ -129,5 +129,5 @@
     <origin xyz="-0.0295 -0.1025 -0.518363" rpy="0 0 0"/>
     <geometry>
-      <mesh filename="$(find FINAL_description)/meshes/Gear_3,_UPDATED_1.stl" scale="0.001 0.001 0.001"/>
+      <mesh filename="package://FINAL_description/meshes/Gear_3,_UPDATED_1.stl" scale="0.001 0.001 0.001"/>
     </geometry>
   </collision>
@@ -142,5 +142,5 @@
     <origin xyz="-0.4145 -0.1025 -0.518363" rpy="0 0 0"/>
     <geometry>
-      <mesh filename="$(find FINAL_description)/meshes/Manipulator3__2__1.stl" scale="0.001 0.001 0.001"/>
+      <mesh filename="package://FINAL_description/meshes/Manipulator3__2__1.stl" scale="0.001 0.001 0.001"/>
     </geometry>
     <material name="grey"/>
@@ -149,5 +149,5 @@
     <origin xyz="-0.4145 -0.1025 -0.518363" rpy="0 0 0"/>
     <geometry>
-      <mesh filename="$(find FINAL_description)/meshes/Manipulator3__2__1.stl" scale="0.001 0.001 0.001"/>
+      <mesh filename="package://FINAL_description/meshes/Manipulator3__2__1.stl" scale="0.001 0.001 0.001"/>
     </geometry>
   </collision>
